File: Kicad/Keyboard.kicad_sch (KiCad schematic)
At the start: 68 parts, among them J1 Power, J2 ext_keys, J3 Keyboard Row, J4 Keyboard Column, J5 Cursor keys, U1 74LS32, U2 74LS32, U3 74LS32, U4 74LS32, U5 74LS32

Commit message: shortened board, correction to link symbol shift to some chars, reversed U4 so it faces the same way as all the other ICs
Connections:
- net at D18.2 (A), U2.4: now also D32.2 (A), D34.2 (A), D36.2 (A), D38.2 (A), D40.2 (A), D45.2 (A), D47.2 (A), D49.2 (A), D51.2 (A)
